Commit message: - Fixed scaling - Moved kelpie_webots into dingo_ws - Made launch file

File: dingo_ws/src/kelpie_webots/webot/klp_urdf/klp.urdf (robot description, URDF)
Before this commit: robot Robot, 13 links, 12 joints
Links:
- link Base: geometry collision mesh filename=meshes\collision\base_coll.stl scale=1 1 1; visual mesh filename=meshes\visual\base.stl scale=0.001 0.001 0.001
- link Body01: geometry collision mesh filename=meshes\collision\Body01_coll.stl scale=1 1 1; visual mesh filename=meshes\visual\Body01.stl scale=0.001 0.001 0.001
- link Body02: geometry collision mesh filename=meshes\collision\Body02_coll.stl scale=1 1 1; visual mesh filename=meshes\visual\Body02.stl scale=0.001 0.001 0.001
- link Body03: geometry collision mesh filename=meshes\collision\Body03_coll.stl scale=1 1 1; visual mesh filename=meshes\visual\Body03.stl scale=0.001 0.001 0.001
- link Body04: geometry collision mesh filename=meshes\collision\Body04_coll.stl scale=1 1 1; visual mesh filename=meshes\visual\Body04.stl scale=0.001 0.001 0.001
- link Body05: geometry collision mesh filename=meshes\collision\Body02_coll.stl scale=1 1 1; visual mesh filename=meshes\visual\Body02.stl scale=0.001 0.001 0.001
- link Body06: geometry collision mesh filename=meshes\collision\Body03_coll.stl scale=1 1 1; visual mesh filename=meshes\visual\Body03.stl scale=0.001 0.001 0.001
- link Body07: geometry collision mesh filename=meshes\collision\Body07_coll.stl scale=1 1 1; visual mesh filename=meshes\visual\Body07.stl scale=0.001 0.001 0.001
- link Body08: geometry collision mesh filename=meshes\collision\Body02_coll.stl scale=1 1 1; visual mesh filename=meshes\visual\Body02.stl scale=0.001 0.001 0.001
- link Body09: geometry collision mesh filename=meshes\collision\Body09_coll.stl scale=1 1 1; visual mesh filename=meshes\visual\Body09.stl scale=0.001 0.001 0.001
- link Body10: geometry collision mesh filename=meshes\collision\Body10_coll.stl scale=1 1 1; visual mesh filename=meshes\visual\Body10.stl scale=0.001 0.001 0.001
- link Body11: geometry collision mesh filename=meshes\collision\Body02_coll.stl scale=1 1 1; visual mesh filename=meshes\visual\Body02.stl scale=0.001 0.001 0.001
- link Body12: geometry collision mesh filename=meshes\collision\Body09_coll.stl scale=1 1 1; visual mesh filename=meshes\visual\Body09.stl scale=0.001 0.001 0.001
