Commit message: Changed scaling of stl files and fixed incorrect urdf/proto lower leg alignments.

File: dingo_ws/src/kelpie_webots/launch/webots/klp_urdf/klp.urdf (robot description, URDF)
Before this commit: robot Robot, 13 links, 12 joints
Links:
- link Base: geometry collision mesh filename=meshes\collision\base_coll.stl scale=1.00000000 1.00000000 1.00000000; visual mesh filename=meshes\visual\base.stl scale=1.00000000 1.00000000 1.00000000
- link Body01: geometry collision mesh filename=meshes\collision\Body01_coll.stl scale=1.00000000 1.00000000 1.00000000; visual mesh filename=meshes\visual\Body01.stl scale=1.00000000 1.00000000 1.00000000
- link Body02: geometry collision mesh filename=meshes\collision\Body02_coll.stl scale=1.00000000 1.00000000 1.00000000; visual mesh filename=meshes\visual\Body02.stl scale=1.00000000 1.00000000 1.00000000
- link Body03: geometry collision mesh filename=meshes\collision\Body03_coll.stl scale=1.00000000 1.00000000 1.00000000; visual mesh filename=meshes\visual\Body03.stl scale=1.00000000 1.00000000 1.00000000
- link Body04: geometry collision mesh filename=meshes\collision\Body04_coll.stl scale=1.00000000 1.00000000 1.00000000; visual mesh filename=meshes\visual\Body04.stl scale=1.00000000 1.00000000 1.00000000
- link Body05: geometry collision mesh filename=meshes\collision\Body02_coll.stl scale=1.00000000 1.00000000 1.00000000; visual mesh filename=meshes\visual\Body02.stl scale=1.00000000 1.00000000 1.00000000
- link Body06: geometry collision mesh filename=meshes\collision\Body03_coll.stl scale=1.00000000 1.00000000 1.00000000; visual mesh filename=meshes\visual\Body03.stl scale=1.00000000 1.00000000 1.00000000
- link Body07: geometry collision mesh filename=meshes\collision\Body07_coll.stl scale=1.00000000 1.00000000 1.00000000; visual mesh filename=meshes\visual\Body07.stl scale=1.00000000 1.00000000 1.00000000
- link Body08: geometry collision mesh filename=meshes\collision\Body02_coll.stl scale=1.00000000 1.00000000 1.00000000; visual mesh filename=meshes\visual\Body02.stl scale=1.00000000 1.00000000 1.00000000
- link Body09: geometry collision mesh filename=meshes\collision\Body09_coll.stl scale=1.00000000 1.00000000 1.00000000; visual mesh filename=meshes\visual\Body09.stl scale=1.00000000 1.00000000 1.00000000
- link Body10: geometry collision mesh filename=meshes\collision\Body10_coll.stl scale=1.00000000 1.00000000 1.00000000; visual mesh filename=meshes\visual\Body10.stl scale=1.00000000 1.00000000 1.00000000
- link Body11: geometry collision mesh filename=meshes\collision\Body02_coll.stl scale=1.00000000 1.00000000 1.00000000; visual mesh filename=meshes\visual\Body02.stl scale=1.00000000 1.00000000 1.00000000
- link Body12: geometry collision mesh filename=meshes\collision\Body09_coll.stl scale=1.00000000 1.00000000 1.00000000; visual mesh filename=meshes\visual\Body09.stl scale=1.00000000 1.00000000 1.00000000
Joints:
- joint Joint03: origin xyz=-0.12987943 -0.00559767 -0.02600000 rpy=3.14159265 0.00000000 0.00000000 -> xyz=-0.12990000  0.00000000 -0.02600000 rpy=3.14159265 0.00000000 0.00000000
- joint Joint06: origin xyz=-0.12987943 -0.00559767 -0.02600000 rpy=3.14159265 0.00000000 0.00000000 -> xyz=-0.12990000  0.00000000 -0.02600000 rpy=3.14159265 0.00000000 0.00000000
- joint Joint09: origin xyz=-0.12987943 -0.00559767 -0.02600000 rpy=3.14159265 0.00000000 0.00000000 -> xyz=-0.12987943  0.00000000 -0.02600000 rpy=3.14159265 0.00000000 0.00000000
- joint Joint12: origin xyz=-0.12987943 -0.00559767 -0.02600000 rpy=3.14159265 0.00000000 0.00000000 -> xyz=-0.12987943  0.00000000 -0.02600000 rpy=3.14159265 0.00000000 0.00000000
